Commit message: Complete-ish demo, add driver app

File: k4a_arm_support/urdf/workcell.xacro (robot description, xacro)
@@ -4,5 +4,5 @@
   <xacro:robotiq_c2_model prefix=""/>
   <xacro:include filename="$(find ur_description)/urdf/ur3.urdf.xacro"/>
-  <xacro:ur3_robot prefix="" joint_limited="true"/>
+  <xacro:ur3_robot prefix="" joint_limited="false"/>
   <link name="world"/>
   <link name="winml_link"/>
@@ -61,5 +61,5 @@
       <parent link="ee_link"/>
       <child link="k_mount"/>
-      <origin xyz="0.0 0.0 0.0" rpy="0.0 0.0 0.0"/>
+      <origin xyz="0.0 0.0 0.0" rpy="${-pi} 0.0 0.0"/>
   </joint>
   <joint name="k_mount_to_k" type="fixed">
