Commit message: use robotiq_arg2f_85 model, and adjust camera geometry.

File: k4a_arm_support/urdf/UR3_Lifecam.xacro (robot description, xacro)
@@ -1,6 +1,6 @@
 <?xml version="1.0" ?>
 <robot name="UR3_with_k4a" xmlns:xacro="http://ros.org/wiki/xacro">
-  <xacro:include filename="$(find robotiq_2f_c2_gripper_visualization)/urdf/robotiq_c2_model_macro.xacro" />
-  <xacro:robotiq_c2_model prefix=""/>
+  <xacro:include filename="$(find robotiq_2f_85_gripper_visualization)/urdf/robotiq_arg2f_85_model_macro.xacro" />
+  <xacro:robotiq_arg2f_85 prefix=""/>
   <xacro:include filename="$(find ur_description)/urdf/ur3.urdf.xacro"/>
   <xacro:ur3_robot prefix="" joint_limited="false"/>
@@ -56,5 +56,5 @@
     <visual>
       <geometry>
-        <cylinder length="0.03" radius="0.015"/>
+        <cylinder length="0.07" radius="0.02"/>
       </geometry>
       <material name="White">
@@ -64,5 +64,5 @@
     <collision>
       <geometry>
-        <cylinder length="0.03" radius="0.015"/>
+        <cylinder length="0.07" radius="0.015"/>
       </geometry>
     </collision>
@@ -95,6 +95,6 @@
   <joint name="k_mount_to_adapter" type="fixed">
       <parent link="k_mount"/>
-      <child link="robotiq_85_adapter_link"/>
-      <origin xyz="0.017 0 0" rpy="0 ${-pi/2} 0"/>
+      <child link="robotiq_arg2f_base_link"/>
+      <origin xyz="0 0 0.02" rpy="0 0 0"/>
   </joint>
   <joint name="winml_to_k4a_optical" type="fixed">

Commit message: correct the optical location.

File: k4a_arm_support/urdf/UR3_Lifecam.xacro (robot description, xacro)
@@ -101,5 +101,5 @@
       <parent link="k4a_link_optical"/>
       <child link="winml_link"/>
-      <origin xyz="0 0 0" rpy="0 0 0"/>
+      <origin xyz="0 0 0.027" rpy="0 0 0"/>
   </joint>
   <joint name="k4a_optical_joint" type="fixed">

Commit message: add aruco marker detect  support.

File: k4a_arm_support/urdf/UR3_Lifecam.xacro (robot description, xacro)
@@ -8,4 +8,64 @@
   <link name="winml_link"/>
   <link name="k4a_link_optical" />
+  <link name="wall1">
+      <visual>
+          <geometry>
+              <box size="1.0 0.05 1.0"/>
+          </geometry>
+          <material name="Green">
+          <color rgba="0.0 0.5 0.0 0.5"/>
+          </material>
+      </visual>
+      <collision>
+          <geometry>
+              <box size="1.0 0.05 1.0"/>
+          </geometry>
+      </collision>
+  </link>
+  <link name="wall2">
+      <visual>
+          <geometry>
+              <box size="1.0 0.05 1.0"/>
+          </geometry>
+          <material name="Green">
+          <color rgba="0.0 0.5 0.0 0.5"/>
+          </material>
+      </visual>
+      <collision>
+          <geometry>
+              <box size="1.0 0.05 1.0"/>
+          </geometry>
+      </collision>
+  </link>
+  <link name="wall3">
+      <visual>
+          <geometry>
+              <box size="1.0 1.0 0.05"/>
+          </geometry>
+          <material name="Green">
+          <color rgba="0.0 0.5 0.0 0.5"/>
+          </material>
+      </visual>
+      <collision>
+          <geometry>
+              <box size="1.0 1.0 0.05"/>
+          </geometry>
+      </collision>
+  </link>
+  <link name="wall4">
+      <visual>
+          <geometry>
+              <box size="0.05 1.0 1.0"/>
+          </geometry>
+          <material name="Green">
+          <color rgba="0.0 0.5 0.0 0.5"/>
+          </material>
+      </visual>
+      <collision>
+          <geometry>
+              <box size="0.05 1.0 1.0"/>
+          </geometry>
+      </collision>
+  </link>
   <link name="table">
       <visual>
@@ -73,4 +133,24 @@
       <origin xyz="0 0 0.0" rpy="0 0 0"/>
   </joint>
+  <joint name="world_to_wall1" type="fixed">
+      <parent link="world"/>
+      <child link="wall1"/>
+      <origin xyz="0 0.3 0.5" rpy="0 0 0"/>
+  </joint>
+  <joint name="world_to_wall2" type="fixed">
+      <parent link="world"/>
+      <child link="wall2"/>
+      <origin xyz="0 -0.3 0.5" rpy="0 0 0"/>
+  </joint>
+  <joint name="world_to_wall3" type="fixed">
+      <parent link="world"/>
+      <child link="wall3"/>
+      <origin xyz="0 0 0.7" rpy="0 0 0"/>
+  </joint>
+  <joint name="world_to_wall4" type="fixed">
+      <parent link="world"/>
+      <child link="wall4"/>
+      <origin xyz="0.3 0 0.5" rpy="0 0 0"/>
+  </joint>
   <joint name="ee_to_k_mount" type="fixed">
       <parent link="ee_link"/>
@@ -86,5 +166,5 @@
       <parent link="table"/>
       <child link="robot_mount"/>
-      <origin xyz="0 0 0.012" rpy="0 0 0"/>
+      <origin xyz="0 0 0.012" rpy="0 0 ${pi/2}"/>
   </joint>
   <joint name="robot_mount_to_robot" type="fixed">
